Commit message: feat(file_server2 + gazebo_simulation_scene2): Remove duplicate and gazebo2 example specific URDF files.

File: ROS Packages/ROS2/file_server2/urdf/custom_r2d2.urdf (robot description, URDF)
Before this commit: robot physics, 16 links, 15 joints
Joints:
- joint gripper_extension: limit lower=-0.38 upper=0 effort=1000.0 velocity=0.5 -> (none); type prismatic -> fixed
