Commit message: fix(gazebo_simulation_scene2): Use exact odometry instead of the estimation from diff drive plugin + correct plane position + update r2d2 urdf with the new odometry plugin

File: com.siemens.ros-sharp/Samples~/Gazebo Simulation Scenes ROS2/Urdf/file_server2/robot_description.urdf (robot description, URDF)
Before this commit: robot r2d2, 11 links, 10 joints
Links:
- added link gripper_pole, mass 0.05; collision cylinder length=0.2 radius=0.01; visual cylinder length=0.2 radius=0.01
- added link left_gripper, mass 0.05; collision mesh filename=package://urdf_tutorial/meshes/l_finger.dae; visual mesh filename=package://urdf_tutorial/meshes/l_finger.dae
- added link left_tip, mass 0.05; collision mesh filename=package://urdf_tutorial/meshes/l_finger_tip.dae; visual mesh filename=package://urdf_tutorial/meshes/l_finger_tip.dae
- added link right_gripper, mass 0.05; collision mesh filename=package://urdf_tutorial/meshes/l_finger.dae; visual mesh filename=package://urdf_tutorial/meshes/l_finger.dae
- added link right_tip, mass 0.05; collision mesh filename=package://urdf_tutorial/meshes/l_finger_tip.dae; visual mesh filename=package://urdf_tutorial/meshes/l_finger_tip.dae
Joints:
- added joint gripper_extension: type fixed, parent base_link, child gripper_pole, origin xyz=0.19 0 0.2 rpy=0 0 0
- added joint left_gripper_joint: type revolute, parent gripper_pole, child left_gripper, origin xyz=0.2 0.01 0 rpy=0 0 0, axis 0 0 1, limit lower=0.0 upper=0.548 effort=1000.0 velocity=0.5
- added joint left_tip_joint: type fixed, parent left_gripper, child left_tip
- added joint right_gripper_joint: type revolute, parent gripper_pole, child right_gripper, origin xyz=0.2 -0.01 0 rpy=0 0 0, axis 0 0 -1, limit lower=0.0 upper=0.548 effort=1000.0 velocity=0.5
- added joint right_tip_joint: type fixed, parent right_gripper, child right_tip
